File: MeccanoidArduinoShield-EAGLE/Board-TODO.brd (EAGLE design)
At the start: 71.1 x 55.5 mm, 27 parts

Commit message: Update content for youtube video
Parts:
- removed D2: 1N4004, diode:DO41-10
- removed DC1+, DC1-, DC2+, DC2-, MECCANOID-VIN, MECCANOID-VIN-GND: (no value), wirepad:1,6/0,8
- removed HM-10, SERVO-5V, SERVO-GND: (no value), pinhead:1X04
- removed K1K2+, K1K2-, K3K4+, K3K4-: (no value), pinhead:1X03/90
- removed LD1, LD2, LD3: (no value), led:LED3MM
- removed R3: 731Ω, resistor:0207/5V
- removed RELAY-ALIM: (no value), pinhead:1X02
- removed S1, S2: (no value), switch:255SB
- removed SERVO-SIGNAL: (no value), pinhead:1X03
- added D10, D3: (no value), diode:DO35-7
- added HM-10-BLUETOOTH: (no value), pinhead:1X04
- added IC2: (no value), arduino:ARDUINO2009
- added LED1, LED2: (no value), pinhead:1X02
- added M1, M2: 308-100, motor:308-100
- added RELAY-OUPUT-A, RELAY-OUTPUT-B, RELAY-OUTPUT-C, RELAY-OUTPUT-D, SERVO-CONTROL: (no value), pinhead:1X03
- D1: value 1N4004 -> (none); device diode:DO41-10 -> diode:DO35-7
- R1, R2: value 731Ω -> (none); device resistor:0207/5V -> resistor:0204V
- RELAY-CONTROL: device pinhead:1X04 -> pinhead:1X06
- moved RELAY-CONTROL 110.1 mm to (55.9, 113.0)
- moved R2 109.0 mm to (11.4, 118.1)
- moved R1 104.1 mm to (16.5, 118.1)
- moved D1 92.5 mm to (58.4, 118.1), turned to 0 degrees
- moved IC1 92.3 mm to (-5.08, 2.54), turned to 0 degrees
Connections:
- removed net N$14: IC1.17, RELAY-CONTROL.3
- removed net N$25: LD3.A, R3.2
- removed net N$26: IC1.22, R3.1
- removed net N$27: IC1.21, R2.1
- removed net N$28: DC2+.1, K3K4+.2, K3K4-.2
- removed net N$29: DC2-.1, K3K4+.1, K3K4-.1
- removed net N$30: IC1.6, K1K2+.3, K3K4+.3, MECCANOID-VIN.1
- removed net N$31: D2.A, IC1.5, K1K2-.3, LD1.K, LD2.K, LD3.K, SERVO-GND.1, SERVO-GND.2, SERVO-GND.3, SERVO-GND.4
- new net +3V3: IC2.2
- new net +5V: D1.A, D1.C, IC2.3, IC2.6, RELAY-OUPUT-A.1, RELAY-OUTPUT-B.1, RELAY-OUTPUT-C.1, RELAY-OUTPUT-D.1
- new net GND: IC1.27, IC2.27, IC2.4, RELAY-OUPUT-A.3, RELAY-OUTPUT-B.3, RELAY-OUTPUT-D.3
- new net N$22: IC2.5, LED1.2, LED2.2
- new net N$8: D3.A, IC1.3
- new net RELAY-OUTPUT-D: M2.NEG, RELAY-OUTPUT-D.2
- net N$1: now also M1.POS, RELAY-OUPUT-A.2; no longer HM-10.3, IC1.4
- net N$10: now also M1.NEG, RELAY-OUTPUT-B.2; no longer IC1.25, SERVO-SIGNAL.2
- net N$11: now also IC2.24, SERVO-CONTROL.1; no longer IC1.24, SERVO-SIGNAL.1
- net N$12: now also D10.C, IC1.5; no longer IC1.15, RELAY-CONTROL.1
- net N$13: now also IC2.25, SERVO-CONTROL.2; no longer IC1.16, RELAY-CONTROL.2
- net N$15: now also IC2.26, SERVO-CONTROL.3; no longer IC1.18, RELAY-CONTROL.4
- net N$16: now also HM-10-BLUETOOTH.1, IC1.2; no longer D2.C, RELAY-ALIM.1
- net N$17: now also D10.A, RELAY-CONTROL.6; no longer IC1.20, R1.1
- net N$18: now also HM-10-BLUETOOTH.2, IC1.13, IC2.13; no longer DC1+.1, K1K2+.2, K1K2-.2
- net N$19: now also HM-10-BLUETOOTH.4, IC1.4; no longer IC1.14, S1.1
- net N$2: now also M2.POS, RELAY-OUTPUT-C.2; no longer HM-10.4, IC1.2
- net N$20: now also HM-10-BLUETOOTH.3, IC1.14, IC2.14; no longer HM-10.1, S1.2
- net N$21: now also LED1.1; no longer LD1.A
- net N$23: now also LED2.1, R2.2; no longer DC1-.1, K1K2+.1, K1K2-.1
- net N$24: now also IC2.20, R2.1; no longer LD2.A, R2.2
- net N$3: now also D3.C, RELAY-CONTROL.1; no longer IC1.13, S2.1
- net N$4: now also IC1.15, RELAY-CONTROL.2; no longer D1.A, IC1.3, SERVO-5V.1, SERVO-5V.2, SERVO-5V.3, SERVO-5V.4
- net N$5: now also IC1.16, RELAY-CONTROL.3; no longer HM-10.2, S2.2
- net N$6: now also IC1.17, RELAY-CONTROL.4; no longer D1.C, RELAY-ALIM.2
- net N$7: now also IC1.18, RELAY-CONTROL.5; no longer IC1.27, MECCANOID-VIN-GND.1
- net N$9: now also IC2.16, R1.1; no longer IC1.26, SERVO-SIGNAL.3
Other:
- board size 71.1 x 55.5 mm -> 160 x 100 mm
